File: UART_peripheral_card_A.sch (KiCad schematic (older format))
At the start: 16 parts, among them J1 PP1_edgeConnnector_TE_5-55308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, J2 power_connector, J3 UART_connector, J4 OUTPUT_MODE, U1 74AHC1G00, U2 74AHC1G00, U27 74AHC1G125, U28 74AHC1G125, U4 74AHC1G00, U5 74AHC1G00

Commit message: netlist, association, CHANGELOG
Parts:
- U1, U2, U4, U5: footprint (none) -> Package_TO_SOT_SMD:SOT-23-5
Changed lines of the file:
@@
 F 0 "U1" H 1850 5350 50  0000 L CNN
 F 1 "74AHC1G00" H 1850 5250 50  0000 L CNN
-F 2 "" H 1700 5100 50  0001 C CNN
+F 2 "Package_TO_SOT_SMD:SOT-23-5" H 1700 5100 50  0001 C CNN
 F 3 "https://assets.nexperia.com/documents/data-sheet/74AHC_AHCT1G00.pdf" H 1700 5100 50  0001 C CNN
 	1    1700 5100
@@
 F 0 "U4" H 3700 5350 50  0000 L CNN
 F 1 "74AHC1G00" H 3700 5250 50  0000 L CNN
-F 2 "" H 3550 5100 50  0001 C CNN
+F 2 "Package_TO_SOT_SMD:SOT-23-5" H 3550 5100 50  0001 C CNN
 F 3 "https://assets.nexperia.com/documents/data-sheet/74AHC_AHCT1G00.pdf" H 3550 5100 50  0001 C CNN
 	1    3550 5100
@@
 F 0 "U5" H 3700 6350 50  0000 L CNN
 F 1 "74AHC1G00" H 3700 6250 50  0000 L CNN
-F 2 "" H 3550 6100 50  0001 C CNN
+F 2 "Package_TO_SOT_SMD:SOT-23-5" H 3550 6100 50  0001 C CNN
 F 3 "https://assets.nexperia.com/documents/data-sheet/74AHC_AHCT1G00.pdf" H 3550 6100 50  0001 C CNN
 	1    3550 6100
@@
 F 0 "U2" H 1850 6350 50  0000 L CNN
 F 1 "74AHC1G00" H 1850 6250 50  0000 L CNN
-F 2 "" H 1700 6100 50  0001 C CNN
+F 2 "Package_TO_SOT_SMD:SOT-23-5" H 1700 6100 50  0001 C CNN
 F 3 "https://assets.nexperia.com/documents/data-sheet/74AHC_AHCT1G00.pdf" H 1700 6100 50  0001 C CNN
 	1    1700 6100
