File: fileReception.sch (KiCad schematic (older format))
At the start: 19 parts, among them U10 74AHC1G00, U11 74AHC1G32, U13 74AHC595, U6 LTC6994xS6-1, U7 LTC6990CS6, U8 CD74AC161M, U9 74HCT107

Commit message: netlist, association, CHANGELOG
Parts:
- U10: footprint (none) -> Package_TO_SOT_SMD:SOT-23-5
Changed lines of the file:
@@
 F 0 "U10" H 4800 6750 50  0000 L CNN
 F 1 "74AHC1G00" H 4800 6650 50  0000 L CNN
-F 2 "" H 4650 6500 50  0001 C CNN
+F 2 "Package_TO_SOT_SMD:SOT-23-5" H 4650 6500 50  0001 C CNN
 F 3 "https://assets.nexperia.com/documents/data-sheet/74AHC_AHCT1G00.pdf" H 4650 6500 50  0001 C CNN
 	1    4650 6500
