File: fileTransmission.sch (KiCad schematic (older format))
At the start: 24 parts, among them U14 74HCT107, U15 CD74AC161M, U16 LTC6990CS6, U17 LTC6994xS6-1, U18 74AHC1G32, U19 74AHC1G32, U20 74AHC1G00, U21 74AHC1G32, U23 74AHC1G04, U24 74AHC1G08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

Commit message: netlist, association, CHANGELOG
Parts:
- U20: footprint (none) -> Package_TO_SOT_SMD:SOT-23-5
Changed lines of the file:
@@
 F 0 "U20" H 4850 4650 50  0000 L CNN
 F 1 "74AHC1G00" H 4850 4550 50  0000 L CNN
-F 2 "" H 4700 4400 50  0001 C CNN
+F 2 "Package_TO_SOT_SMD:SOT-23-5" H 4700 4400 50  0001 C CNN
 F 3 "https://assets.nexperia.com/documents/data-sheet/74AHC_AHCT1G00.pdf" H 4700 4400 50  0001 C CNN
 	1    4700 4400
